File: TechLab AVR DevBoard.kicad_sch (KiCad schematic)
At the start: 258 parts, among them IC1 ATMEGA32A-PU, IC2 PCF8583T_5,518, J1 Conn_01x01, J10 Screw_Terminal_01x02, J11 1761682-3, J12 Screw_Terminal_01x02, J13 Conn_01x02, J14 Conn_01x02, J15 Conn_01x02, J16 Conn_01x03, J17 Conn_01x02, J18 Conn_01x02, J19 Screw_Terminal_01x02, J2 Conn_02x08_Odd_Even, J20 Screw_Terminal_01x02, J21 Screw_Terminal_01x02, J22 Screw_Terminal_01x02, J23 USB_B, J24 Conn_01x02, J25 Conn_01x01, J26 Conn_01x02, J27 Conn_01x08, J28 Conn_01x02, J29 Conn_01x02, J3 Conn_01x03, J30 Conn_01x01, J31 Conn_01x02, J32 Conn_01x08, J33 Conn_01x08, J34 Conn_01x08, J35 Conn_01x03, J36 Conn_01x01, J37 Conn_01x01, J38 Screw_Terminal_01x02, J39 Conn_02x05_Odd_Even, J4 Conn_01x16, J40 Conn_01x02, J41 Conn_01x04, J42 Conn_01x03, J43 Conn_01x03, J44 Conn_01x01, J45 Conn_01x03, J46 Conn_01x02, J47 Conn_01x02, J48 Conn_01x04, J49 Screw_Terminal_01x02, J5 Conn_01x02, J50 Screw_Terminal_01x02, J51 Screw_Terminal_01x02, J52 Conn_01x04, J53 Conn_01x02, J6 Conn_01x08, J7 Conn_01x02, J8 Conn_01x08, J9 Screw_Terminal_01x02, Q1 BC817W, Q2 BC807, Q3 LTV-355T, Q4 LTV-355T, Q5 BC817W, Q6 BC807, Q7 BC807, Q8 BC807, Q9 BC807, SW1 SW_DIP_x02, SW10 SW_Push_Dual_x2, SW11 SW_Push_Dual_x2, SW12 SW_Push_Dual_x2, SW13 SW_Push_Dual_x2, SW14 SW_Push_Dual_x2, SW15 SW_Push_Dual_x2, SW2 SW_DIP_x01, SW3 SW_DIP_x02, SW4 RotaryEncoder_Switch, SW5 SW_DIP_x02, SW6 SW_DIP_x01, SW7 SW_DIP_x01, SW8 SW_DIP_x01, SW9 SW_DIP_x01, U1 IFX27001TFV33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

Commit message: V2023.1
Parts:
- removed U4: TSOP312xx, OptoDevice:Vishay_CAST-3Pin, symbol Interface_Optical:TSOP312xx
- added BT1: Battery_Cell, Battery:BatteryHolder_Keystone_103_1x20mm, symbol Device:Battery_Cell
- added H10, H9: MountingHole, MountingHole:MountingHole_2.2mm_M2_ISO7380, symbol Mechanical:MountingHole
- added H11: MountingHole, MountingHole:MountingHole_3.5mm_Pad_Via, symbol Mechanical:MountingHole
- added H5, H6, H7, H8: MountingHole, MountingHole:MountingHole_3.2mm_M3_ISO14580, symbol Mechanical:MountingHole
- added IR1, IR2: Conn_01x03, Connector_PinHeader_2.54mm:PinHeader_1x03_P2.54mm_Vertical, symbol Connector_Generic:Conn_01x03
- added IR3: Conn_01x04, Connector_PinSocket_2.54mm:PinSocket_1x04_P2.54mm_Vertical, symbol Connector_Generic:Conn_01x04
- added J54: Conn_01x02, Connector_PinHeader_2.54mm:PinHeader_1x02_P2.54mm_Vertical, symbol Connector_Generic:Conn_01x02
- D2, D3, D4, D5: footprint LED_SMD:LED_0603_1608Metric -> LED_SMD:LED_0805_2012Metric
- D6: footprint Diode_SMD:D_SOD-123 -> Diode_THT:D_DO-35_SOD27_P7.62mm_Horizontal
- VR1: footprint PTN10E10SB20 -> TechLab:PTN10E10SB20
- VR2: footprint P120PKY25BR10K -> TechLab:P120PKY25BR10K
Connections:
- net GND: now also BT1.2 (-), IR1.3 (Pin_3), IR2.2 (Pin_2), IR3.1 (Pin_1)
- net VCC: now also S2.3 (NO); no longer SelPwrSrc1.2 (Pin_2)
- net at S2.2 (COM): now also SelPwrSrc1.2 (Pin_2); no longer D1.1 (K)
- net at C4.2, J16.1 (Pin_1): now also D1.1 (K); no longer S2.3 (NO)
- net at C24.1, R18.1: now also IR1.2 (Pin_2), IR2.3 (Pin_3), IR3.2 (Pin_2)
- net at D18.2: now also J54.2 (Pin_2)
- net at R17.1, SW2.2: now also IR1.1 (Pin_1), IR2.1 (Pin_1), IR3.4 (Pin_4)
- new net: BT1.1 (+), J54.1 (Pin_1)
Other:
- moved on the sheet: D6, Ovr33Reg1, R16, S2, vcc1
